File: rev2/ecad/IV_variation.kicad_sch (KiCad schematic)
At the start: 35 parts, among them Q1 IRF3205, Q2 IRF4905, Q5 IRF3205, Q6 IRF4905, U2 LM6144xIx

Commit message: restructuring and layout
Parts:
- D2: footprint (none) -> Diode_THT:D_DO-15_P10.16mm_Horizontal
- F?: footprint (none) -> Fuse:Fuse_1206_3216Metric_Pad1.42x1.75mm_HandSolder
- HS1, HS2, HS3, HS4: value 577202B00000G -> 24.40°C/W
- R10, R19: value 51.1k -> 250k
- R16: value 10k -> 10k+/-0.1%
- TP1, TP2, TP3, TP4, TP5, TP6: footprint (none) -> TestPoint:TestPoint_THTPad_D2.5mm_Drill1.2mm
- U2: footprint (none) -> Package_DIP:DIP-14_W7.62mm
Other:
- moved on the sheet: C8, C?, D2, F?, HS1, HS2, HS3, HS4, Q1, Q2, Q5, Q6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

Commit message: layout
Parts:
- added D3, D4, D5: BZX79-C4V7, Diode_THT:D_DO-35_SOD27_P7.62mm_Horizontal, symbol Device:D_Zener
- added R23, R28, R29, R30, R5: 1k, Resistor_THT:R_Axial_DIN0207_L6.3mm_D2.5mm_P7.62mm_Horizontal, symbol Device:R_US
- D2: value SA6.5CA -> SA13CA
- R10, R19: value 250k -> 250k+/-0.1%
- R14, R17: value 4.02k -> 10k+/-0.1%
- R15, R18, R8: value 10k -> 10k+/-0.1%
- R20: value 10k -> 1k
- R? (x2): value 4.02k -> 1k
- R?: value 0.1 -> 0.1+/-0.1%
- U2: value LM6144xIx -> MCP604
Connections:
- net DUT+: now also R6.2; no longer R20.2
- net DUT_I: now also D4.1 (K), R23.2, R28.1; no longer R19.2, U2.14
- net DUT_V: now also R20.1, D3.1 (K), R5.2; no longer R14.2, U2.8
- net GND: now also R20.2, D3.2 (A), D4.2 (A), D5.2 (A), R28.2, R30.2
- net V/2: now also R29.1
- new net: R19.2, R23.1, U2.14
- new net: R14.2, R5.1, U2.8
- new net V/4: D5.1 (K), R29.2, R30.1
Other:
- title: Analog IV Variation -> Analog Front End
- moved on the sheet: C8, C?, D2, F?, HS1, HS2, HS3, HS4, Q1, Q2, Q5, Q6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

Commit message: BOM
Parts:
- HS1, HS2, HS3, HS4: value 24.40°C/W -> 15.60°C/W
Changed lines of the file:
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@@
       (effects (font (size 1.27 1.27)) (justify left))
     )
-    (property "Value" "24.40°C/W" (at 118.11 48.8823 90)
+    (property "Value" "15.60°C/W" (at 118.11 48.8823 90)
       (effects (font (size 1.27 1.27)) (justify left))
     )
@@
       (effects (font (size 1.27 1.27)) (justify left))
     )
-    (property "Value" "24.40°C/W" (at 118.11 36.1823 90)
+    (property "Value" "15.60°C/W" (at 118.11 36.1823 90)
       (effects (font (size 1.27 1.27)) (justify left))
     )
@@
       (effects (font (size 1.27 1.27)) (justify left))
     )
-    (property "Value" "24.40°C/W" (at 105.41 161.9123 90)
+    (property "Value" "15.60°C/W" (at 105.41 161.9123 90)
       (effects (font (size 1.27 1.27)) (justify left))
     )
@@
       (effects (font (size 1.27 1.27)) (justify left))
     )
-    (property "Value" "24.40°C/W" (at 105.41 149.2123 90)
-      (effects (font (size 1.27 1.27)) (justify left))
-    )
+    (property "Value" "15.60°C/W" (at 105.41 149.2123 90)
+      (effects (font (size 1.27 1.27)) (justify left))
+    )

Commit message: removed ignored files
Parts:
- D3, D4: value BZX79-C4V7 -> BZX79-C2V4
- R5: value 1k -> 2k
- U2: value MCP604 -> MCP6044
Changed lines of the file:
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@@
       (effects (font (size 1.27 1.27)))
     )
-    (property "Value" "MCP604" (at 186.69 120.65 0)
+    (property "Value" "MCP6044" (at 186.69 120.65 0)
       (effects (font (size 1.27 1.27)))
     )
@@
       (effects (font (size 1.27 1.27)))
     )
-    (property "Value" "MCP604" (at 72.39 34.29 0)
+    (property "Value" "MCP6044" (at 72.39 34.29 0)
       (effects (font (size 1.27 1.27)))
     )
@@
       (effects (font (size 1.27 1.27)) (justify left))
     )
-    (property "Value" "MCP604" (at 57.15 148.59 0)
+    (property "Value" "MCP6044" (at 57.15 148.59 0)
       (effects (font (size 1.27 1.27)) (justify left))
     )
@@
       (effects (font (size 1.27 1.27)))
     )
-    (property "Value" "MCP604" (at 62.23 158.75 0)
+    (property "Value" "MCP6044" (at 62.23 158.75 0)
       (effects (font (size 1.27 1.27)))
     )
@@
       (effects (font (size 1.27 1.27)) (justify left))
     )
-    (property "Value" "BZX79-C4V7" (at 237.49 93.345 90)
+    (property "Value" "BZX79-C2V4" (at 237.49 93.345 90)
       (effects (font (size 1.27 1.27)) (justify left))
     )
@@
       (effects (font (size 1.27 1.27)))
     )
-    (property "Value" "MCP604" (at 193.04 69.85 0)
+    (property "Value" "MCP6044" (at 193.04 69.85 0)
       (effects (font (size 1.27 1.27)))
     )
@@
       (effects (font (size 1.27 1.27)) (justify left))
     )
-    (property "Value" "1k" (at 227.33 83.185 0)
+    (property "Value" "2k" (at 227.33 83.185 0)
       (effects (font (size 1.27 1.27)) (justify left))
     )
@@
       (effects (font (size 1.27 1.27)) (justify left))
     )
-    (property "Value" "BZX79-C4V7" (at 232.41 144.145 90)
-      (effects (font (size 1.27 1.27)) (justify left))
-    )
+    (property "Value" "BZX79-C2V4" (at 232.41 144.145 90)
+      (effects (font (size 1.27 1.27)) (justify left))
+    )

Commit message: Linear Output
Parts:
- removed Q1, Q5: IRF3205, Package_TO_SOT_THT:TO-220-3_Vertical, symbol Transistor_FET:IRF3205
- removed Q2, Q6: IRF4905, Package_TO_SOT_THT:TO-220-3_Vertical, symbol Transistor_FET:IRF4905
- added Q1, Q5: TIP122, Package_TO_SOT_THT:TO-220-3_Vertical, symbol Transistor_BJT:TIP122
- added Q2, Q6: TIP127, Package_TO_SOT_THT:TO-220-3_Vertical, symbol Transistor_BJT:TIP127
- D5: value BZX79-C4V7 -> BZX79-C2V4
- R18, R8: value 10k+/-0.1% -> 1k
- R23: value 1k -> 3240
- R29: value 1k -> 4.7k
- R5: value 2k -> 4.7k
- U2: value MCP6044 -> LM324
Connections:
- net +12V: now also Q1.2 (C), Q5.2 (C)
- net DUT+: now also Q5.3 (E), Q6.3 (E)
- net GND: now also Q2.2 (C), Q6.2 (C)
- net V/2: now also Q1.3 (E), Q2.3 (E)
- net at R?.2: now also Q5.1 (B), Q6.1 (B)
- net at R?.2: now also Q1.1 (B), Q2.1 (B)
- net V/4 renamed Vmiddle
