File: rev2/ecad/USB_curve_tracer.kicad_pcb (KiCad board)
At the start: 2 copper layers, 111 x 64 mm, 58 parts, among them J1 DUT Connector, J2 Power Input, Q1 IRF3205, Q2 IRF4905, Q5 IRF3205, Q6 IRF4905, U1 MCP4911, U2 LM6144xIx, U3 MCP3204, U4 LM285Z-2.5

Commit message: layout
Parts:
- added D3: BZX79-C4V7, Diode_THT:D_DO-35_SOD27_P7.62mm_Horizontal, F.Cu at (148.1, 84.0)
- added D4: BZX79-C4V7, Diode_THT:D_DO-35_SOD27_P7.62mm_Horizontal, F.Cu at (150.6, 120.4)
- added D5: BZX79-C4V7, Diode_THT:D_DO-35_SOD27_P7.62mm_Horizontal, F.Cu at (158.3, 96.8)
- added R23: 1k, Resistor_THT:R_Axial_DIN0207_L6.3mm_D2.5mm_P7.62mm_Horizontal, F.Cu at (158.4, 113.0)
- added R28: 1k, Resistor_THT:R_Axial_DIN0207_L6.3mm_D2.5mm_P7.62mm_Horizontal, F.Cu at (150.8, 109.8)
- added R29: 1k, Resistor_THT:R_Axial_DIN0207_L6.3mm_D2.5mm_P7.62mm_Horizontal, F.Cu at (150.7, 103.1)
- added R30: 1k, Resistor_THT:R_Axial_DIN0207_L6.3mm_D2.5mm_P7.62mm_Horizontal, F.Cu at (158.3, 99.9)
- added R5: 1k, Resistor_THT:R_Axial_DIN0207_L6.3mm_D2.5mm_P7.62mm_Horizontal, F.Cu at (151.2, 76.4)
- D2: value SA6.5CA -> SA13CA
- R10, R19: value 250k -> 250k+/-0.1%
- R13: value 0.1 -> 0.1+/-0.1%
- R14, R17: value 4.02k -> 10k+/-0.1%
- R15, R18, R8: value 10k -> 10k+/-0.1%
- R20: value 10k -> 1k
- R4, R9: value 4.02k -> 1k
- U2: value LM6144xIx -> MCP604
- moved TP4 41.0 mm to (145.2, 72.7)
- moved R20 36.9 mm to (154.5, 84.0)
- moved TP5 19.6 mm to (140.8, 114.5)
- moved F1 13.2 mm to (97.9, 114.8)
- moved R21 12.4 mm to (174.7, 84.0), turned to 90 degrees
- moved C2 11.1 mm to (174.7, 72.0), turned to 180 degrees
- moved C8 11.0 mm to (122.3, 111.6)
- moved Q2 11.0 mm to (132.1, 74.4)
- moved Q6 11.0 mm to (132.1, 120.4)
- moved R13 11.0 mm to (140.9, 88.1)
- moved R18 11.0 mm to (141.0, 94.7)
- moved R19 11.0 mm to (141.0, 91.5)
- moved R8 11.0 mm to (141.0, 98.0)
- moved TP2 11.0 mm to (141.0, 77.0)
- moved U2 11.0 mm to (122.3, 92.4)
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Connections:
- R14 pad 2: /IV_Variation/DUT_V -> Net-(R14-Pad2)
- R19 pad 2: /IV_Variation/DUT_I -> Net-(R19-Pad2)
- R20 pad 1: Net-(R20-Pad1) -> /IV_Variation/DUT_V
- R20 pad 2: /IV_Variation/DUT+ -> GND
- R6 pad 2: Net-(R20-Pad1) -> /IV_Variation/DUT+
- U2 pad 14: /IV_Variation/DUT_I -> Net-(R19-Pad2)
- U2 pad 8: /IV_Variation/DUT_V -> Net-(R14-Pad2)
- U3 pad 3: V/2 -> /IV_Variation/V/4
Routing:
- net Net-(R19-Pad2): track 0.00 -> 58.7 mm, vias 0 -> 2
- net Net-(R14-Pad2): track 0.00 -> 54.4 mm, vias 0 -> 3
- net +12V: track 137.9 -> 176.2 mm
- net /IV_Variation/DUT+: track 146.9 -> 125.8 mm, vias 4 -> 2
- net /IV_Variation/DUT_V: track 55.6 -> 35.2 mm
- net V/2: track 105.7 -> 126.0 mm, vias 0 -> 2
- net /IV_Variation/DUT_I: track 37.4 -> 57.7 mm, vias 2 -> 0
- net Net-(U2C-+): track 18.5 -> 37.4 mm
- net +5V: track 0.00 -> 16.1 mm, vias 0 -> 6
- net Net-(A1-D10): track 54.2 -> 67.4 mm
- net /IV_Variation/V/4: track 0.00 -> 11.8 mm
- net /IV_Variation/VADJ: track 69.5 -> 81.3 mm, vias 7 -> 8
- net Net-(U2D-+): track 17.2 -> 26.4 mm
- net Net-(U3-Vref): track 30.3 -> 23.1 mm
- net /IV_Variation/DUT-: track 96.3 -> 101.0 mm
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Other:
- board size 111 x 64 mm -> 117 x 64 mm
- board text removed: "FIX THE FUCKING GRID SNAP ISSUE"

Commit message: BOM
Parts:
- U4: value LM285Z-2.5 -> LM385BZ-2.5
Other:
- board text added: "Curve Tracer"
- board text added: "MN"
- board text added: "REV2"
Changed lines of the file:
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@@
         (effects (font (size 1 1) (thickness 0.15)))
     )
-    (fp_text value "LM285Z-2.5" (at 1.27 2.79) (layer "F.Fab")
+    (fp_text value "LM385BZ-2.5" (at 1.27 2.79) (layer "F.Fab")
         (effects (font (size 1 1) (thickness 0.15)))
     )
@@
     (effects (font (size 1 1) (thickness 0.15)) (justify left bottom))
   )
+  (gr_text "MN" (at 190 132) (layer "F.SilkS")
+    (effects (font (size 1 1) (thickness 0.15)) (justify left bottom))
+  )
+  (gr_text "REV2" (at 102 132) (layer "F.SilkS")
+    (effects (font (size 1 1) (thickness 0.15)) (justify left bottom))
+  )
   (gr_text "DUT+" (at 94.500169 95.053452) (layer "F.SilkS")
     (effects (font (size 1 1) (thickness 0.15)) (justify left bottom))
@@
     (effects (font (size 1 1) (thickness 0.15)) (justify left bottom))
   )
+  (gr_text "Curve Tracer" (at 91 132) (layer "F.SilkS")
+    (effects (font (size 1 1) (thickness 0.15)) (justify left bottom))
+  )

Commit message: removed ignored files
Parts:
- D3, D4: value BZX79-C4V7 -> BZX79-C2V4
- R5: value 1k -> 2k
- U2: value MCP604 -> MCP6044
Changed lines of the file:
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@@
         (effects (font (size 1 1) (thickness 0.15)))
     )
-    (fp_text value "BZX79-C4V7" (at 3.81 2.12 90) (layer "F.Fab")
+    (fp_text value "BZX79-C2V4" (at 3.81 2.12 90) (layer "F.Fab")
         (effects (font (size 1 1) (thickness 0.15)))
     )
@@
         (effects (font (size 1 1) (thickness 0.15)))
     )
-    (fp_text value "BZX79-C4V7" (at 3.81 2.12) (layer "F.Fab")
+    (fp_text value "BZX79-C2V4" (at 3.81 2.12) (layer "F.Fab")
         (effects (font (size 1 1) (thickness 0.15)))
     )
@@
         (effects (font (size 1 1) (thickness 0.15)))
     )
-    (fp_text value "1k" (at 3.81 2.37 90) (layer "F.Fab")
+    (fp_text value "2k" (at 3.81 2.37 90) (layer "F.Fab")
         (effects (font (size 1 1) (thickness 0.15)))
     )
@@
     (property "ki_keywords" "12bit ADC Reference Single Supply SPI 4ch")
     (attr through_hole)
-    (fp_text reference "U3" (at 3.81 -2.33) (layer "F.SilkS")
+    (fp_text reference "U3" (at -0.197056 -2.187944) (layer "F.SilkS")
         (effects (font (size 1 1) (thickness 0.15)))
     )
@@
     (fp_line (start 1.6 0.8) (end -1.6 0.8)
       (stroke (width 0.1) (type solid)) (layer "F.Fab"))
-    (pad "1" smd roundrect (at -1.4875 0) (size 1.425 1.75) (layers "F.Cu" "F.Paste" "F.Mask") (roundrect_rratio 0.175439)
+    (pad "1" smd roundrect (at -1.4875 0) (size 1.425 1.75) (layers "F.Cu" "F.Paste" "F.Mask") (roundrect_rratio 0.1754392982)
       (net 36 "Net-(J2-Pin_2)") (pintype "passive"))
-    (pad "2" smd roundrect (at 1.4875 0) (size 1.425 1.75) (layers "F.Cu" "F.Paste" "F.Mask") (roundrect_rratio 0.175439)
+    (pad "2" smd roundrect (at 1.4875 0) (size 1.425 1.75) (layers "F.Cu" "F.Paste" "F.Mask") (roundrect_rratio 0.1754392982)
       (net 16 "+12V") (pintype "passive"))
     (model "${KICAD6_3DMODEL_DIR}/Fuse.3dshapes/Fuse_1206_3216Metric.wrl"
@@
     (fp_line (start 1.6 0.8) (end -1.6 0.8)
       (stroke (width 0.1) (type solid)) (layer "F.Fab"))
-    (pad "1" smd roundrect (at -1.4875 0) (size 1.425 1.75) (layers "F.Cu" "F.Paste" "F.Mask") (roundrect_rratio 0.175439)
+    (pad "1" smd roundrect (at -1.4875 0) (size 1.425 1.75) (layers "F.Cu" "F.Paste" "F.Mask") (roundrect_rratio 0.1754392982)
       (net 32 "/IV_Variation/DUT-") (pintype "passive"))
-    (pad "2" smd roundrect (at 1.4875 0) (size 1.425 1.75) (layers "F.Cu" "F.Paste" "F.Mask") (roundrect_rratio 0.175439)
+    (pad "2" smd roundrect (at 1.4875 0) (size 1.425 1.75) (layers "F.Cu" "F.Paste" "F.Mask") (roundrect_rratio 0.1754392982)
       (net 37 "Net-(F2-Pad2)") (pintype "passive"))
     (model "${KICAD6_3DMODEL_DIR}/Fuse.3dshapes/Fuse_1206_3216Metric.wrl"
@@
         (effects (font (size 1 1) (thickness 0.15)))
     )
-    (fp_text value "MCP604" (at 3.81 17.57) (layer "F.Fab")
+    (fp_text value "MCP6044" (at 3.81 17.57) (layer "F.Fab")
         (effects (font (size 1 1) (thickness 0.15)))
     )

Commit message: Linear Output
Parts:
- D1: value SA6.0A -> SA13A
- D5: value BZX79-C4V7 -> BZX79-C2V4
- Q1, Q5: value IRF3205 -> TIP122
- Q2, Q6: value IRF4905 -> TIP127
- R23: value 1k -> 3240
- R29: value 1k -> 4.7k
- R5: value 2k -> 4.7k
- U2: value MCP6044 -> LMC6484IN
Connections:
- net /IV_Variation/V/4 renamed /IV_Variation/Vmiddle
