File: electronics/rev3/ecad/USB_curve_tracer.kicad_sch (KiCad schematic)
At the start: 27 parts, among them J1 DUT Connector, J2 Power Input, U1 MCP4911, U3 MCP3204, U4 LM385BZ-2.5

Commit message: REV3 schematic
Parts:
- removed J1: DUT Connector, TerminalBlock_Phoenix:TerminalBlock_Phoenix_MKDS-1,5-2-5.08_1x02_P5.08mm_Horizontal, symbol Connector:Screw_Terminal_01x02
- C1, C2, C5: Distributor Part # (none) -> BC2665CT-ND; Part # (none) -> K104K10X7RF5UH5; Unit Price (none) -> 0.23
- C3: Distributor Part # (none) -> 445-173437-1-ND; Part # (none) -> FG26X7R1E106KRT06; Unit Price (none) -> 0.65
- D1: Distributor Part # (none) -> SA13A-E3/54GICT-ND; Part # (none) -> SA13A-E3/54; Unit Price (none) -> 0.46
- D6: Distributor Part # (none) -> 754-1735-ND; Part # (none) -> WP7113SGD; Unit Price (none) -> 0.34
- D7: Distributor Part # (none) -> 754-1264-ND; Part # (none) -> WP7113ID; Unit Price (none) -> 0.1
- F1: value 2A -> 3A; Distributor Part # (none) -> 507-1896-1-ND; Part # (none) -> 0685T3000-01; Unit Price (none) -> 0.32
- J2: Distributor Part # (none) -> 102-6179-ND; Part # (none) -> TB004-508-02BE; Unit Price (none) -> 0.71
- R1, R22, R24, R25, R26, R27: Distributor Part # (none) -> CF14JT10K0CT-ND; Part # (none) -> CF14JT10K0; Unit Price (none) -> 0.1
- R11, R12: Distributor Part # (none) -> 619XBK-ND; Part # (none) -> MFR-25FBF52-619R; Unit Price (none) -> 0.1
Connections:
- net IV_Variation/VADJ renamed IV_Variation/Sweep_Input
Other:
- sheet IV_Variation ports: added Sweep_Input; removed DUT+, DUT-, VADJ
- moved on the sheet: C2, R21, R22

Commit message: Layout work
Parts:
- added D16: 1N5817, Diode_THT:D_DO-41_SOD81_P10.16mm_Horizontal, symbol Diode:1N5817
- H1, H2, H3, H4: Distributor Part # (none) -> HS351-ND; Part # (none) -> 531002B02500G; Unit Price (none) -> 1.55
- R21: Distributor Part # (none) -> 14.0KXBK-ND; Part # (none) -> MFR-25FBF52-14K; Unit Price (none) -> 0.1
- U1: Distributor Part # (none) -> MCP4911-E/P-ND; Part # (none) -> MCP4911-E/P; Unit Price (none) -> 1.97
- U3: Distributor Part # (none) -> MCP3204-CI/P-ND; Part # (none) -> MCP3204-CI/P; Unit Price (none) -> 4.52
- U4: Distributor Part # (none) -> LM385BZ-2.5GOS-ND; Part # (none) -> LM385BZ-2.5G; Unit Price (none) -> 0.78
Connections:
- net +12V: now also D16.1 (K); no longer F1.2
- new net: D16.2 (A), F1.2
Other:
- moved on the sheet: C3, D1, H1, H2, H3, H4

Commit message: start direction modes
Parts:
- A1: Distributor Part # (none) -> 1050-ABX00033-ND; Part # (none) -> ABX00033; Unit Price (none) -> 14.91
- D16: Distributor Part # (none) -> 497-4547-1-ND; Part # (none) -> 1N5817; Unit Price (none) -> 0.44
Changed lines of the file:
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@@
   (title_block
     (title "USB Curve Tracer")
-    (date "2023-09-27")
+    (date "2023-10-10")
     (rev "3")
     (comment 1 "Designed by Marek Newton")
@@
       (effects (font (size 1.27 1.27)) hide)
     )
+    (property "Distributor Part #" "497-4547-1-ND" (at 64.77 166.37 0)
+      (effects (font (size 1.27 1.27)) hide)
+    )
+    (property "Part #" "1N5817" (at 64.77 166.37 0)
+      (effects (font (size 1.27 1.27)) hide)
+    )
+    (property "Unit Price" "0.44" (at 64.77 166.37 0)
+      (effects (font (size 1.27 1.27)) hide)
+    )
     (pin "1")
     (pin "2")
@@
       (effects (font (size 1.27 1.27)) hide)
     )
-    (property "Distributor Part #" "" (at 224.79 99.06 0)
-      (effects (font (size 1.27 1.27)) hide)
-    )
-    (property "Part #" "" (at 224.79 99.06 0)
-      (effects (font (size 1.27 1.27)) hide)
-    )
-    (property "Unit Price" "" (at 224.79 99.06 0)
-      (effects (font (size 1.27 1.27)) hide)
-    )
+    (property "Distributor Part #" "1050-ABX00033-ND" (at 224.79 99.06 0)
+      (effects (font (size 1.27 1.27)) hide)
+    )
+    (property "Part #" "ABX00033" (at 224.79 99.06 0)
+      (effects (font (size 1.27 1.27)) hide)
+    )
+    (property "Unit Price" "14.91" (at 224.79 99.06 0)
+      (effects (font (size 1.27 1.27)) hide)
+    )

Commit message: value changes
Parts:
- D7: value WP7113ID -> XLUR12D
- R21: value 14k -> 16.2k
Changed lines of the file:
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@@
   (symbol (lib_id "Device:R_US") (at 195.58 80.01 0) (unit 1)
     (in_bom yes) (on_board yes) (dnp no) (fields_autoplaced)
-    (property "Reference" "R21" (at 198.12 79.375 0)
+    (property "Reference" "R21" (at 198.12 78.74 0)
       (effects (font (size 1.27 1.27)) (justify left))
     )
-    (property "Value" "14k" (at 198.12 81.915 0)
+    (property "Value" "16.2k" (at 198.12 81.28 0)
       (effects (font (size 1.27 1.27)) (justify left))
     )
@@
       (effects (font (size 1.27 1.27)))
     )
-    (property "Value" "WP7113ID" (at 240.03 147.32 0)
+    (property "Value" "XLUR12D" (at 240.03 147.32 0)
       (effects (font (size 1.27 1.27)))
     )
