File: electronics/rev3/ecad/IV_variation.kicad_sch (KiCad schematic)
At the start: 31 parts, among them J1 DUT Connector, U2 LMC6484A

Commit message: added tolerance
Parts:
- R30: value 1k -> 1k+/-0.1%
Other:
- moved on the sheet: C10, D5
Changed lines of the file:
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@@
   (junction (at 120.65 139.7) (diameter 0) (color 0 0 0 0)
   )
-  (junction (at 144.78 157.48) (diameter 0) (color 0 0 0 0)
+  (junction (at 153.67 157.48) (diameter 0) (color 0 0 0 0)
   )
   (junction (at 120.65 140.97) (diameter 0) (color 0 0 0 0)
@@
   (junction (at 120.65 157.48) (diameter 0) (color 0 0 0 0)
   )
-  (junction (at 134.62 157.48) (diameter 0) (color 0 0 0 0)
+  (junction (at 143.51 157.48) (diameter 0) (color 0 0 0 0)
   )
   (junction (at 214.63 127) (diameter 0) (color 0 0 0 0)
@@
     (stroke (width 0) (type default))
   )
-  (wire (pts (xy 144.78 157.48) (xy 147.32 157.48))
+  (wire (pts (xy 153.67 157.48) (xy 156.21 157.48))
     (stroke (width 0) (type default))
   )
@@
     (stroke (width 0) (type default))
   )
-  (wire (pts (xy 134.62 157.48) (xy 144.78 157.48))
+  (wire (pts (xy 143.51 157.48) (xy 153.67 157.48))
     (stroke (width 0) (type default))
   )
@@
     (stroke (width 0) (type default))
   )
-  (wire (pts (xy 134.62 166.37) (xy 134.62 167.64))
+  (wire (pts (xy 143.51 166.37) (xy 143.51 167.64))
     (stroke (width 0) (type default))
   )
@@
     (stroke (width 0) (type default))
   )
-  (wire (pts (xy 144.78 166.37) (xy 144.78 167.64))
+  (wire (pts (xy 153.67 166.37) (xy 153.67 167.64))
     (stroke (width 0) (type default))
   )
@@
     (stroke (width 0) (type default))
   )
-  (wire (pts (xy 120.65 157.48) (xy 134.62 157.48))
+  (wire (pts (xy 120.65 157.48) (xy 143.51 157.48))
     (stroke (width 0) (type default))
   )
@@
     (stroke (width 0) (type default))
   )
-  (wire (pts (xy 144.78 157.48) (xy 144.78 158.75))
+  (wire (pts (xy 153.67 157.48) (xy 153.67 158.75))
     (stroke (width 0) (type default))
   )
@@
     (stroke (width 0) (type default))
   )
-  (wire (pts (xy 134.62 157.48) (xy 134.62 158.75))
+  (wire (pts (xy 143.51 157.48) (xy 143.51 158.75))
     (stroke (width 0) (type default))
   )
@@
     (effects (font (size 1.27 1.27)) (justify left))
   )
-  (hierarchical_label "Vmiddle" (shape output) (at 147.32 157.48 0) (fields_autoplaced)
+  (hierarchical_label "Vmiddle" (shape output) (at 156.21 157.48 0) (fields_autoplaced)
     (effects (font (size 1.27 1.27)) (justify left))
   )
@@
     )
   )
-  (symbol (lib_id "power:GND") (at 144.78 167.64 0) (mirror y) (unit 1)
-    (in_bom yes) (on_board yes) (dnp no) (fields_autoplaced)
-    (property "Reference" "#PWR?" (at 144.78 173.99 0)
-      (effects (font (size 1.27 1.27)) hide)
-    )
-    (property "Value" "GND" (at 144.78 172.72 0)
-      (effects (font (size 1.27 1.27)))
-    )
-    (property "Footprint" "" (at 144.78 167.64 0)
-      (effects (font (size 1.27 1.27)) hide)
-    )
-    (property "Datasheet" "" (at 144.78 167.64 0)
+  (symbol (lib_id "power:GND") (at 153.67 167.64 0) (mirror y) (unit 1)
+    (in_bom yes) (on_board yes) (dnp no) (fields_autoplaced)
+    (property "Reference" "#PWR?" (at 153.67 173.99 0)
+      (effects (font (size 1.27 1.27)) hide)
+    )
+    (property "Value" "GND" (at 153.67 172.72 0)
+      (effects (font (size 1.27 1.27)))
+    )
+    (property "Footprint" "" (at 153.67 167.64 0)
+      (effects (font (size 1.27 1.27)) hide)
+    )
+    (property "Datasheet" "" (at 153.67 167.64 0)
       (effects (font (size 1.27 1.27)) hide)
     )
@@
       (effects (font (size 1.27 1.27)) (justify left))
     )
-    (property "Value" "1k" (at 123.19 163.83 0)
+    (property "Value" "1k+/-0.1%" (at 123.19 163.83 0)
       (effects (font (size 1.27 1.27)) (justify left))
     )
@@
     )
   )
-  (symbol (lib_id "power:GND") (at 134.62 167.64 0) (mirror y) (unit 1)
-    (in_bom yes) (on_board yes) (dnp no) (fields_autoplaced)
-    (property "Reference" "#PWR?" (at 134.62 173.99 0)
-      (effects (font (size 1.27 1.27)) hide)
-    )
-    (property "Value" "GND" (at 134.62 172.72 0)
-      (effects (font (size 1.27 1.27)))
-    )
-    (property "Footprint" "" (at 134.62 167.64 0)
-      (effects (font (size 1.27 1.27)) hide)
-    )
-    (property "Datasheet" "" (at 134.62 167.64 0)
+  (symbol (lib_id "power:GND") (at 143.51 167.64 0) (mirror y) (unit 1)
+    (in_bom yes) (on_board yes) (dnp no) (fields_autoplaced)
+    (property "Reference" "#PWR?" (at 143.51 173.99 0)
+      (effects (font (size 1.27 1.27)) hide)
+    )
+    (property "Value" "GND" (at 143.51 172.72 0)
+      (effects (font (size 1.27 1.27)))
+    )
+    (property "Footprint" "" (at 143.51 167.64 0)
+      (effects (font (size 1.27 1.27)) hide)
+    )
+    (property "Datasheet" "" (at 143.51 167.64 0)
       (effects (font (size 1.27 1.27)) hide)
     )
@@
     )
   )
-  (symbol (lib_id "Device:D_Zener") (at 144.78 162.56 270) (unit 1)
+  (symbol (lib_id "Device:D_Zener") (at 153.67 162.56 270) (unit 1)
     (in_bom yes) (on_board yes) (dnp no)
-    (property "Reference" "D5" (at 147.32 160.02 90)
-      (effects (font (size 1.27 1.27)) (justify left))
-    )
-    (property "Value" "BZX79-C2V4" (at 147.32 162.56 90)
-      (effects (font (size 1.27 1.27)) (justify left))
-    )
-    (property "Footprint" "Diode_THT:D_DO-35_SOD27_P7.62mm_Horizontal" (at 144.78 162.56 0)
-      (effects (font (size 1.27 1.27)) hide)
-    )
-    (property "Datasheet" "~" (at 144.78 162.56 0)
-      (effects (font (size 1.27 1.27)) hide)
-    )
-    (property "Distributor Part #" "1727-2115-1-ND" (at 144.78 162.56 0)
-      (effects (font (size 1.27 1.27)) hide)
-    )
-    (property "Part #" "BZX79-C2V4,113" (at 144.78 162.56 0)
-      (effects (font (size 1.27 1.27)) hide)
-    )
-    (property "Unit Price" "0.16" (at 144.78 162.56 0)
+    (property "Reference" "D5" (at 156.21 160.02 90)
+      (effects (font (size 1.27 1.27)) (justify left))
+    )
+    (property "Value" "BZX79-C2V4" (at 156.21 162.56 90)
+      (effects (font (size 1.27 1.27)) (justify left))
+    )
+    (property "Footprint" "Diode_THT:D_DO-35_SOD27_P7.62mm_Horizontal" (at 153.67 162.56 0)
+      (effects (font (size 1.27 1.27)) hide)
+    )
+    (property "Datasheet" "~" (at 153.67 162.56 0)
+      (effects (font (size 1.27 1.27)) hide)
+    )
+    (property "Distributor Part #" "1727-2115-1-ND" (at 153.67 162.56 0)
+      (effects (font (size 1.27 1.27)) hide)
+    )
+    (property "Part #" "BZX79-C2V4,113" (at 153.67 162.56 0)
+      (effects (font (size 1.27 1.27)) hide)
+    )
+    (property "Unit Price" "0.16" (at 153.67 162.56 0)
       (effects (font (size 1.27 1.27)) hide)
     )
@@
     )
   )
-  (symbol (lib_id "Device:C") (at 134.62 162.56 0) (unit 1)
+  (symbol (lib_id "Device:C") (at 143.51 162.56 0) (unit 1)
     (in_bom yes) (on_board yes) (dnp no)
-    (property "Reference" "C10" (at 137.16 161.29 0)
-      (effects (font (size 1.27 1.27)) (justify left))
-    )
-    (property "Value" "0.1uF" (at 137.16 163.83 0)
-      (effects (font (size 1.27 1.27)) (justify left))
-    )
-    (property "Footprint" "Capacitor_THT:C_Disc_D6.0mm_W2.5mm_P5.00mm" (at 135.5852 166.37 0)
-      (effects (font (size 1.27 1.27)) hide)
-    )
-    (property "Datasheet" "~" (at 134.62 162.56 0)
-      (effects (font (size 1.27 1.27)) hide)
-    )
-    (property "Distributor Part #" "BC2665CT-ND" (at 134.62 162.56 0)
-      (effects (font (size 1.27 1.27)) hide)
-    )
-    (property "Part #" "K104K10X7RF5UH5" (at 134.62 162.56 0)
-      (effects (font (size 1.27 1.27)) hide)
-    )
-    (property "Unit Price" "0.23" (at 134.62 162.56 0)
-      (effects (font (size 1.27 1.27)) hide)
-    )
+    (property "Reference" "C10" (at 146.05 161.29 0)
+      (effects (font (size 1.27 1.27)) (justify left))
+    )
+    (property "Value" "0.1uF" (at 146.05 163.83 0)
+      (effects (font (size 1.27 1.27)) (justify left))
+    )
+    (property "Footprint" "Capacitor_THT:C_Disc_D6.0mm_W2.5mm_P5.00mm" (at 144.4752 166.37 0)
+      (effects (font (size 1.27 1.27)) hide)
+    )
+    (property "Datasheet" "~" (at 143.51 162.56 0)
+      (effects (font (size 1.27 1.27)) hide)
+    )
+    (property "Distributor Part #" "BC2665CT-ND" (at 143.51 162.56 0)
+      (effects (font (size 1.27 1.27)) hide)
+    )
+    (property "Part #" "K104K10X7RF5UH5" (at 143.51 162.56 0)
+      (effects (font (size 1.27 1.27)) hide)
+    )
+    (property "Unit Price" "0.23" (at 143.51 162.56 0)
+      (effects (font (size 1.27 1.27)) hide)
+    )

Commit message: removed zener diodes
Parts:
- removed D3, D4, D5: BZX79-C2V4, Diode_THT:D_DO-35_SOD27_P7.62mm_Horizontal, symbol Device:D_Zener
Changed lines of the file:
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@@
   (junction (at 120.65 139.7) (diameter 0) (color 0 0 0 0)
   )
-  (junction (at 153.67 157.48) (diameter 0) (color 0 0 0 0)
-  )
   (junction (at 120.65 140.97) (diameter 0) (color 0 0 0 0)
   )
@@
   (junction (at 120.65 130.81) (diameter 0) (color 0 0 0 0)
   )
-  (junction (at 217.17 62.23) (diameter 0) (color 0 0 0 0)
-  )
   (junction (at 214.63 62.23) (diameter 0) (color 0 0 0 0)
   )
   (junction (at 102.87 140.97) (diameter 0) (color 0 0 0 0)
   )
-  (junction (at 217.17 127) (diameter 0) (color 0 0 0 0)
-  )
   (junction (at 158.75 49.53) (diameter 0) (color 0 0 0 0)
   )
@@
     (stroke (width 0) (type default))
   )
-  (wire (pts (xy 214.63 127) (xy 217.17 127))
-    (stroke (width 0) (type default))
-  )
   (wire (pts (xy 120.65 77.47) (xy 143.51 77.47))
     (stroke (width 0) (type default))
@@
     (stroke (width 0) (type default))
   )
-  (wire (pts (xy 153.67 157.48) (xy 156.21 157.48))
+  (wire (pts (xy 143.51 157.48) (xy 156.21 157.48))
     (stroke (width 0) (type default))
   )
@@
     (stroke (width 0) (type default))
   )
-  (wire (pts (xy 217.17 127) (xy 219.71 127))
-    (stroke (width 0) (type default))
-  )
-  (wire (pts (xy 143.51 157.48) (xy 153.67 157.48))
+  (wire (pts (xy 214.63 127) (xy 219.71 127))
     (stroke (width 0) (type default))
   )
@@
     (stroke (width 0) (type default))
   )
-  (wire (pts (xy 217.17 135.89) (xy 217.17 137.16))
-    (stroke (width 0) (type default))
-  )
   (wire (pts (xy 120.65 64.77) (xy 120.65 68.58))
     (stroke (width 0) (type default))
@@
     (stroke (width 0) (type default))
   )
-  (wire (pts (xy 153.67 166.37) (xy 153.67 167.64))
-    (stroke (width 0) (type default))
-  )
   (wire (pts (xy 129.54 129.54) (xy 129.54 130.81))
     (stroke (width 0) (type default))
@@
     (stroke (width 0) (type default))
   )
-  (wire (pts (xy 217.17 62.23) (xy 218.44 62.23))
-    (stroke (width 0) (type default))
-  )
-  (wire (pts (xy 217.17 127) (xy 217.17 128.27))
-    (stroke (width 0) (type default))
-  )
   (wire (pts (xy 182.88 115.57) (xy 185.42 115.57))
     (stroke (width 0) (type default))
@@
     (stroke (width 0) (type default))
   )
-  (wire (pts (xy 153.67 157.48) (xy 153.67 158.75))
-    (stroke (width 0) (type default))
-  )
   (wire (pts (xy 157.48 59.69) (xy 158.75 59.69))
     (stroke (width 0) (type default))
@@
     (stroke (width 0) (type default))
   )
-  (wire (pts (xy 214.63 62.23) (xy 217.17 62.23))
+  (wire (pts (xy 214.63 62.23) (xy 218.44 62.23))
     (stroke (width 0) (type default))
   )
@@
     (stroke (width 0) (type default))
   )
-  (wire (pts (xy 217.17 72.39) (xy 217.17 71.12))
-    (stroke (width 0) (type default))
-  )
   (wire (pts (xy 156.21 113.03) (xy 167.64 113.03))
     (stroke (width 0) (type default))
@@
   )
   (wire (pts (xy 156.21 121.92) (xy 156.21 123.19))
-    (stroke (width 0) (type default))
-  )
-  (wire (pts (xy 217.17 63.5) (xy 217.17 62.23))
     (stroke (width 0) (type default))
   )
@@
     )
   )
-  (symbol (lib_id "power:GND") (at 217.17 72.39 0) (mirror y) (unit 1)
-    (in_bom yes) (on_board yes) (dnp no) (fields_autoplaced)
-    (property "Reference" "#PWR?" (at 217.17 78.74 0)
-      (effects (font (size 1.27 1.27)) hide)
-    )
-    (property "Value" "GND" (at 217.17 77.47 0)
-      (effects (font (size 1.27 1.27)))
-    )
-    (property "Footprint" "" (at 217.17 72.39 0)
-      (effects (font (size 1.27 1.27)) hide)
-    )
-    (property "Datasheet" "" (at 217.17 72.39 0)
-      (effects (font (size 1.27 1.27)) hide)
-    )
-    (pin "1")
-    (instances
-      (project "USB_curve_tracer"
-        (path "/e63e39d7-6ac0-4ffd-8aa3-1841a4541b55"
-          (reference "#PWR?") (unit 1)
-        )
-        (path "/e63e39d7-6ac0-4ffd-8aa3-1841a4541b55/934ae8eb-860a-4c99-952a-5338d2d71b19"
-          (reference "#PWR036") (unit 1)
-        )
-      )
-    )
-  )
   (symbol (lib_id "Device:R_US") (at 151.13 113.03 90) (unit 1)
     (in_bom yes) (on_board yes) (dnp no)
@@
     )
   )
-  (symbol (lib_id "power:GND") (at 153.67 167.64 0) (mirror y) (unit 1)
-    (in_bom yes) (on_board yes) (dnp no) (fields_autoplaced)
-    (property "Reference" "#PWR?" (at 153.67 173.99 0)
-      (effects (font (size 1.27 1.27)) hide)
-    )
-    (property "Value" "GND" (at 153.67 172.72 0)
-      (effects (font (size 1.27 1.27)))
-    )
-    (property "Footprint" "" (at 153.67 167.64 0)
-      (effects (font (size 1.27 1.27)) hide)
-    )
-    (property "Datasheet" "" (at 153.67 167.64 0)
-      (effects (font (size 1.27 1.27)) hide)
-    )
-    (pin "1")
-    (instances
-      (project "USB_curve_tracer"
-        (path "/e63e39d7-6ac0-4ffd-8aa3-1841a4541b55"
-          (reference "#PWR?") (unit 1)
-        )
-        (path "/e63e39d7-6ac0-4ffd-8aa3-1841a4541b55/934ae8eb-860a-4c99-952a-5338d2d71b19"
-          (reference "#PWR039") (unit 1)
-        )
-      )
-    )
-  )
   (symbol (lib_id "Device:R_US") (at 114.3 39.37 90) (unit 1)
     (in_bom yes) (on_board yes) (dnp no)
@@
         (path "/e63e39d7-6ac0-4ffd-8aa3-1841a4541b55/934ae8eb-860a-4c99-952a-5338d2d71b19"
           (reference "R13") (unit 1)
-        )
-      )
-    )
-  )
-  (symbol (lib_id "Device:D_Zener") (at 217.17 67.31 270) (unit 1)
-    (in_bom yes) (on_board yes) (dnp no) (fields_autoplaced)
-    (property "Reference" "D3" (at 219.71 66.04 90)
-      (effects (font (size 1.27 1.27)) (justify left))
-    )
-    (property "Value" "BZX79-C2V4" (at 219.71 68.58 90)
-      (effects (font (size 1.27 1.27)) (justify left))
-    )
-    (property "Footprint" "Diode_THT:D_DO-35_SOD27_P7.62mm_Horizontal" (at 217.17 67.31 0)
-      (effects (font (size 1.27 1.27)) hide)
-    )
-    (property "Datasheet" "~" (at 217.17 67.31 0)
-      (effects (font (size 1.27 1.27)) hide)
-    )
-    (property "Distributor Part #" "1727-2115-1-ND" (at 217.17 67.31 0)
-      (effects (font (size 1.27 1.27)) hide)
-    )
-    (property "Part #" "BZX79-C2V4,113" (at 217.17 67.31 0)
-      (effects (font (size 1.27 1.27)) hide)
-    )
-    (property "Unit Price" "0.16" (at 217.17 67.31 0)
-      (effects (font (size 1.27 1.27)) hide)
-    )
-    (pin "1")
-    (pin "2")
-    (instances
-      (project "USB_curve_tracer"
-        (path "/e63e39d7-6ac0-4ffd-8aa3-1841a4541b55/934ae8eb-860a-4c99-952a-5338d2d71b19"
-          (reference "D3") (unit 1)
         )
       )
@@
     )
   )
-  (symbol (lib_id "power:GND") (at 217.17 137.16 0) (mirror y) (unit 1)
-    (in_bom yes) (on_board yes) (dnp no) (fields_autoplaced)
-    (property "Reference" "#PWR?" (at 217.17 143.51 0)
-      (effects (font (size 1.27 1.27)) hide)
-    )
-    (property "Value" "GND" (at 217.17 142.24 0)
-      (effects (font (size 1.27 1.27)))
-    )
-    (property "Footprint" "" (at 217.17 137.16 0)
-      (effects (font (size 1.27 1.27)) hide)
-    )
-    (property "Datasheet" "" (at 217.17 137.16 0)
-      (effects (font (size 1.27 1.27)) hide)
-    )
-    (pin "1")
-    (instances
-      (project "USB_curve_tracer"
-        (path "/e63e39d7-6ac0-4ffd-8aa3-1841a4541b55"
-          (reference "#PWR?") (unit 1)
-        )
-        (path "/e63e39d7-6ac0-4ffd-8aa3-1841a4541b55/934ae8eb-860a-4c99-952a-5338d2d71b19"
-          (reference "#PWR038") (unit 1)
-        )
-      )
-    )
-  )
-  (symbol (lib_id "Device:D_Zener") (at 153.67 162.56 270) (unit 1)
-    (in_bom yes) (on_board yes) (dnp no)
-    (property "Reference" "D5" (at 156.21 160.02 90)
-      (effects (font (size 1.27 1.27)) (justify left))
-    )
-    (property "Value" "BZX79-C2V4" (at 156.21 162.56 90)
-      (effects (font (size 1.27 1.27)) (justify left))
-    )
-    (property "Footprint" "Diode_THT:D_DO-35_SOD27_P7.62mm_Horizontal" (at 153.67 162.56 0)
-      (effects (font (size 1.27 1.27)) hide)
-    )
-    (property "Datasheet" "~" (at 153.67 162.56 0)
-      (effects (font (size 1.27 1.27)) hide)
-    )
-    (property "Distributor Part #" "1727-2115-1-ND" (at 153.67 162.56 0)
-      (effects (font (size 1.27 1.27)) hide)
-    )
-    (property "Part #" "BZX79-C2V4,113" (at 153.67 162.56 0)
-      (effects (font (size 1.27 1.27)) hide)
-    )
-    (property "Unit Price" "0.16" (at 153.67 162.56 0)
-      (effects (font (size 1.27 1.27)) hide)
-    )
-    (pin "1")
-    (pin "2")
-    (instances
-      (project "USB_curve_tracer"
-        (path "/e63e39d7-6ac0-4ffd-8aa3-1841a4541b55/934ae8eb-860a-4c99-952a-5338d2d71b19"
-          (reference "D5") (unit 1)
-        )
-      )
-    )
-  )
   (symbol (lib_id "Connector:TestPoint") (at 143.51 69.85 0) (unit 1)
     (in_bom yes) (on_board yes) (dnp no) (fields_autoplaced)
@@
         )
       )
-    )
-  )
-  (symbol (lib_id "Device:D_Zener") (at 217.17 132.08 270) (unit 1)
-    (in_bom yes) (on_board yes) (dnp no) (fields_autoplaced)
-    (property "Reference" "D4" (at 219.71 131.445 90)
-      (effects (font (size 1.27 1.27)) (justify left))
-    )
-    (property "Value" "BZX79-C2V4" (at 219.71 133.985 90)
-      (effects (font (size 1.27 1.27)) (justify left))
-    )
-    (property "Footprint" "Diode_THT:D_DO-35_SOD27_P7.62mm_Horizontal" (at 217.17 132.08 0)
-      (effects (font (size 1.27 1.27)) hide)
-    )
-    (property "Datasheet" "~" (at 217.17 132.08 0)
-      (effects (font (size 1.27 1.27)) hide)
-    )
-    (property "Distributor Part #" "1727-2115-1-ND" (at 217.17 132.08 0)
-      (effects (font (size 1.27 1.27)) hide)
-    )
-    (property "Part #" "BZX79-C2V4,113" (at 217.17 132.08 0)
-      (effects (font (size 1.27 1.27)) hide)
-    )
-    (property "Unit Price" "0.16" (at 217.17 132.08 0)
-      (effects (font (size 1.27 1.27)) hide)
-    )
-    (pin "1")
-    (pin "2")
-    (instances
-      (project "USB_curve_tracer"
-        (path "/e63e39d7-6ac0-4ffd-8aa3-1841a4541b55/934ae8eb-860a-4c99-952a-5338d2d71b19"
-          (reference "D4") (unit 1)
-        )
-      )
