File: electronics/rev3/ecad/half_supply_buffer.kicad_sch (KiCad schematic)
At the start: 19 parts, among them Q1 TIP122, Q2 TIP127, U2 LMC6484A

Commit message: Layout work
Parts:
- HS3, HS4: value 15.60°C/W -> 13.40°C/W; footprint (none) -> Library:HSINK_531002B02500G; Distributor Part # (none) -> HS351-ND; Part # (none) -> 531002B02500G; Unit Price (none) -> 1.55
- TP2: Distributor Part # (none) -> 36-4952-ND; Part # (none) -> 4952; Unit Price (none) -> 0.26
- U2: Distributor Part # (none) -> LMC6484IN/NOPB-ND; Part # (none) -> LMC6484IN/NOPB; Unit Price (none) -> 2.83
Changed lines of the file:
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@@
   )
   (symbol (lib_id "Mechanical:Heatsink") (at 167.64 109.22 270) (unit 1)
-    (in_bom yes) (on_board no) (dnp no) (fields_autoplaced)
-    (property "Reference" "HS4" (at 172.72 108.5723 90)
-      (effects (font (size 1.27 1.27)) (justify left))
-    )
-    (property "Value" "15.60°C/W" (at 172.72 111.1123 90)
-      (effects (font (size 1.27 1.27)) (justify left))
-    )
-    (property "Footprint" "" (at 167.64 109.5248 0)
+    (in_bom yes) (on_board yes) (dnp no) (fields_autoplaced)
+    (property "Reference" "HS4" (at 172.72 107.9373 90)
+      (effects (font (size 1.27 1.27)) (justify left))
+    )
+    (property "Value" "13.40°C/W" (at 172.72 110.4773 90)
+      (effects (font (size 1.27 1.27)) (justify left))
+    )
+    (property "Footprint" "Library:HSINK_531002B02500G" (at 167.64 109.5248 0)
       (effects (font (size 1.27 1.27)) hide)
     )
@@
       (effects (font (size 1.27 1.27)) hide)
     )
-    (property "Distributor Part #" "" (at 167.64 109.22 0)
-      (effects (font (size 1.27 1.27)) hide)
-    )
-    (property "Part #" "" (at 167.64 109.22 0)
-      (effects (font (size 1.27 1.27)) hide)
-    )
-    (property "Unit Price" "" (at 167.64 109.22 0)
+    (property "Distributor Part #" "HS351-ND" (at 167.64 109.22 0)
+      (effects (font (size 1.27 1.27)) hide)
+    )
+    (property "Part #" "531002B02500G" (at 167.64 109.22 0)
+      (effects (font (size 1.27 1.27)) hide)
+    )
+    (property "Unit Price" "1.55" (at 167.64 109.22 0)
       (effects (font (size 1.27 1.27)) hide)
     )
@@
   )
   (symbol (lib_id "Mechanical:Heatsink") (at 168.91 66.04 270) (unit 1)
-    (in_bom yes) (on_board no) (dnp no) (fields_autoplaced)
-    (property "Reference" "HS3" (at 173.99 65.3923 90)
-      (effects (font (size 1.27 1.27)) (justify left))
-    )
-    (property "Value" "15.60°C/W" (at 173.99 67.9323 90)
-      (effects (font (size 1.27 1.27)) (justify left))
-    )
-    (property "Footprint" "" (at 168.91 66.3448 0)
+    (in_bom yes) (on_board yes) (dnp no) (fields_autoplaced)
+    (property "Reference" "HS3" (at 173.99 64.7573 90)
+      (effects (font (size 1.27 1.27)) (justify left))
+    )
+    (property "Value" "13.40°C/W" (at 173.99 67.2973 90)
+      (effects (font (size 1.27 1.27)) (justify left))
+    )
+    (property "Footprint" "Library:HSINK_531002B02500G" (at 168.91 66.3448 0)
       (effects (font (size 1.27 1.27)) hide)
     )
@@
       (effects (font (size 1.27 1.27)) hide)
     )
-    (property "Distributor Part #" "" (at 168.91 66.04 0)
-      (effects (font (size 1.27 1.27)) hide)
-    )
-    (property "Part #" "" (at 168.91 66.04 0)
-      (effects (font (size 1.27 1.27)) hide)
-    )
-    (property "Unit Price" "" (at 168.91 66.04 0)
+    (property "Distributor Part #" "HS351-ND" (at 168.91 66.04 0)
+      (effects (font (size 1.27 1.27)) hide)
+    )
+    (property "Part #" "531002B02500G" (at 168.91 66.04 0)
+      (effects (font (size 1.27 1.27)) hide)
+    )
+    (property "Unit Price" "1.55" (at 168.91 66.04 0)
       (effects (font (size 1.27 1.27)) hide)
     )
@@
       (effects (font (size 1.27 1.27)) hide)
     )
-    (property "Distributor Part #" "" (at 109.22 87.63 0)
-      (effects (font (size 1.27 1.27)) hide)
-    )
-    (property "Part #" "" (at 109.22 87.63 0)
-      (effects (font (size 1.27 1.27)) hide)
-    )
-    (property "Unit Price" "" (at 109.22 87.63 0)
+    (property "Distributor Part #" "LMC6484IN/NOPB-ND" (at 109.22 87.63 0)
+      (effects (font (size 1.27 1.27)) hide)
+    )
+    (property "Part #" "LMC6484IN/NOPB" (at 109.22 87.63 0)
+      (effects (font (size 1.27 1.27)) hide)
+    )
+    (property "Unit Price" "2.83" (at 109.22 87.63 0)
       (effects (font (size 1.27 1.27)) hide)
     )
@@
       (effects (font (size 1.27 1.27)) hide)
     )
-    (property "Distributor Part #" "" (at 187.96 86.36 0)
-      (effects (font (size 1.27 1.27)) hide)
-    )
-    (property "Part #" "" (at 187.96 86.36 0)
-      (effects (font (size 1.27 1.27)) hide)
-    )
-    (property "Unit Price" "" (at 187.96 86.36 0)
+    (property "Distributor Part #" "36-4952-ND" (at 187.96 86.36 0)
+      (effects (font (size 1.27 1.27)) hide)
+    )
+    (property "Part #" "4952" (at 187.96 86.36 0)
+      (effects (font (size 1.27 1.27)) hide)
+    )
+    (property "Unit Price" "0.26" (at 187.96 86.36 0)
       (effects (font (size 1.27 1.27)) hide)
     )
@@
       (effects (font (size 1.27 1.27)) hide)
     )
-    (property "Distributor Part #" "" (at 109.22 87.63 0)
-      (effects (font (size 1.27 1.27)) hide)
-    )
-    (property "Part #" "" (at 109.22 87.63 0)
-      (effects (font (size 1.27 1.27)) hide)
-    )
-    (property "Unit Price" "" (at 109.22 87.63 0)
-      (effects (font (size 1.27 1.27)) hide)
-    )
+    (property "Distributor Part #" "LMC6484IN/NOPB-ND" (at 109.22 87.63 0)
+      (effects (font (size 1.27 1.27)) hide)
+    )
+    (property "Part #" "LMC6484IN/NOPB" (at 109.22 87.63 0)
+      (effects (font (size 1.27 1.27)) hide)
+    )
+    (property "Unit Price" "2.83" (at 109.22 87.63 0)
+      (effects (font (size 1.27 1.27)) hide)
+    )

Commit message: changed crossover resistor to 330
Parts:
- R32: value 1k -> 330
Changed lines of the file:
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@@
       (effects (font (size 1.27 1.27)))
     )
-    (property "Value" "1k" (at 152.4 90.17 90)
+    (property "Value" "330" (at 152.4 90.17 90)
       (effects (font (size 1.27 1.27)))
     )

Commit message: debug and misc
Parts:
- R33: value 10k -> 100k
Changed lines of the file:
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@@
       (effects (font (size 1.27 1.27)))
     )
-    (property "Value" "10k" (at 144.78 143.51 90)
+    (property "Value" "100k" (at 144.78 143.51 90)
       (effects (font (size 1.27 1.27)))
     )
