File: electronics/rev3/ecad/sweep_voltage_buffer.kicad_sch (KiCad schematic)
At the start: 19 parts, among them Q1 TIP122, Q2 TIP127, U2 LMC6484A

Commit message: REV3 schematic
Parts:
- removed C8, C?: 0.1uF, Capacitor_THT:C_Disc_D6.0mm_W2.5mm_P5.00mm, symbol Device:C
- removed C9: 100pF, Capacitor_THT:C_Disc_D6.0mm_W2.5mm_P5.00mm, symbol Device:C
- removed D10, D11, D8, D9: 1N4148, Diode_THT:D_DO-35_SOD27_P7.62mm_Horizontal, symbol Diode:1N4148
- removed HS3, HS4: 15.60°C/W, symbol Mechanical:Heatsink
- removed Q1: TIP122, Package_TO_SOT_THT:TO-220-3_Vertical, symbol Transistor_BJT:TIP122
- removed Q2: TIP127, Package_TO_SOT_THT:TO-220-3_Vertical, symbol Transistor_BJT:TIP127
- removed R31, R4: 4.7k, Resistor_THT:R_Axial_DIN0207_L6.3mm_D2.5mm_P7.62mm_Horizontal, symbol Device:R_US
- removed R32: 1k, Resistor_THT:R_Axial_DIN0207_L6.3mm_D2.5mm_P7.62mm_Horizontal, symbol Device:R_US
- removed R33, R? (x2): 10k, Resistor_THT:R_Axial_DIN0207_L6.3mm_D2.5mm_P7.62mm_Horizontal, symbol Device:R_US
- removed TP2: 4952, TestPoint:TestPoint_THTPad_D2.5mm_Drill1.2mm, symbol Connector:TestPoint
- removed U2: LMC6484A, Package_DIP:DIP-14_W7.62mm, symbol Amplifier_Operational:LM6144xIx
- added C11: 100pF, Capacitor_THT:C_Disc_D6.0mm_W2.5mm_P5.00mm, symbol Device:C
- added D12, D13, D14, D15: 1N4148, Diode_THT:D_DO-35_SOD27_P7.62mm_Horizontal, symbol Diode:1N4148
- added HS1, HS2: 15.60°C/W, symbol Mechanical:Heatsink
- added Q5: TIP122, Package_TO_SOT_THT:TO-220-3_Vertical, symbol Transistor_BJT:TIP122
- added Q6: TIP127, Package_TO_SOT_THT:TO-220-3_Vertical, symbol Transistor_BJT:TIP127
- added R34, R35: 4.7k, Resistor_THT:R_Axial_DIN0207_L6.3mm_D2.5mm_P7.62mm_Horizontal, symbol Device:R_US
- added R6, R7: 10k, Resistor_THT:R_Axial_DIN0207_L6.3mm_D2.5mm_P7.62mm_Horizontal, symbol Device:R_US
- added R9: 1k, Resistor_THT:R_Axial_DIN0207_L6.3mm_D2.5mm_P7.62mm_Horizontal, symbol Device:R_US
- added TP6: TestPoint, TestPoint:TestPoint_THTPad_D2.5mm_Drill1.2mm, symbol Connector:TestPoint
- added U2: LMC6484A, Package_DIP:DIP-14_W7.62mm, symbol Amplifier_Operational:LM6144xIx
Connections:
- net +12V: now also Q5.2 (C), R34.1
- net GND: now also Q6.2 (C), R35.2, R7.2
- new net: C11.2, R6.1, R7.1, U2.2 (-)
- new net: C11.1, D12.1 (K), D14.2 (A), R9.1, U2.1
- new net: D12.2 (A), D13.1 (K)
- new net: D13.2 (A), Q5.1 (B), R34.2
- new net: D15.1 (K), Q6.1 (B), R35.1
- new net: D14.1 (K), D15.2 (A)
- new net Sweep_Amplified: Q5.3 (E), Q6.3 (E), R6.2, R9.2
- new net Sweep_Input: TP6.1, U2.3 (+)
Other:
- title: Half Supply Buffer -> Sweep Voltage Buffer

Commit message: Layout work
Parts:
- HS1, HS2: value 15.60°C/W -> 13.40°C/W; footprint (none) -> Library:HSINK_531002B02500G; Distributor Part # (none) -> HS351-ND; Part # (none) -> 531002B02500G; Unit Price (none) -> 1.55
- TP6: value TestPoint -> 4952; Distributor Part # (none) -> 36-4952-ND; Part # (none) -> 4952; Unit Price (none) -> 0.26
- U2: Distributor Part # (none) -> LMC6484IN/NOPB-ND; Part # (none) -> LMC6484IN/NOPB; Unit Price (none) -> 2.83
Changed lines of the file:
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@@
   )
   (symbol (lib_id "Mechanical:Heatsink") (at 165.1 66.04 270) (unit 1)
-    (in_bom yes) (on_board no) (dnp no) (fields_autoplaced)
-    (property "Reference" "HS2" (at 170.18 65.3923 90)
-      (effects (font (size 1.27 1.27)) (justify left))
-    )
-    (property "Value" "15.60°C/W" (at 170.18 67.9323 90)
-      (effects (font (size 1.27 1.27)) (justify left))
-    )
-    (property "Footprint" "" (at 165.1 66.3448 0)
+    (in_bom yes) (on_board yes) (dnp no) (fields_autoplaced)
+    (property "Reference" "HS2" (at 170.18 64.7573 90)
+      (effects (font (size 1.27 1.27)) (justify left))
+    )
+    (property "Value" "13.40°C/W" (at 170.18 67.2973 90)
+      (effects (font (size 1.27 1.27)) (justify left))
+    )
+    (property "Footprint" "Library:HSINK_531002B02500G" (at 165.1 66.3448 0)
       (effects (font (size 1.27 1.27)) hide)
     )
@@
       (effects (font (size 1.27 1.27)) hide)
     )
-    (property "Distributor Part #" "" (at 165.1 66.04 0)
-      (effects (font (size 1.27 1.27)) hide)
-    )
-    (property "Part #" "" (at 165.1 66.04 0)
-      (effects (font (size 1.27 1.27)) hide)
-    )
-    (property "Unit Price" "" (at 165.1 66.04 0)
+    (property "Distributor Part #" "HS351-ND" (at 165.1 66.04 0)
+      (effects (font (size 1.27 1.27)) hide)
+    )
+    (property "Part #" "531002B02500G" (at 165.1 66.04 0)
+      (effects (font (size 1.27 1.27)) hide)
+    )
+    (property "Unit Price" "1.55" (at 165.1 66.04 0)
       (effects (font (size 1.27 1.27)) hide)
     )
@@
   )
   (symbol (lib_id "Mechanical:Heatsink") (at 163.83 106.68 270) (unit 1)
-    (in_bom yes) (on_board no) (dnp no) (fields_autoplaced)
-    (property "Reference" "HS1" (at 168.91 106.0323 90)
-      (effects (font (size 1.27 1.27)) (justify left))
-    )
-    (property "Value" "15.60°C/W" (at 168.91 108.5723 90)
-      (effects (font (size 1.27 1.27)) (justify left))
-    )
-    (property "Footprint" "" (at 163.83 106.9848 0)
+    (in_bom yes) (on_board yes) (dnp no) (fields_autoplaced)
+    (property "Reference" "HS1" (at 168.91 105.3973 90)
+      (effects (font (size 1.27 1.27)) (justify left))
+    )
+    (property "Value" "13.40°C/W" (at 168.91 107.9373 90)
+      (effects (font (size 1.27 1.27)) (justify left))
+    )
+    (property "Footprint" "Library:HSINK_531002B02500G" (at 163.83 106.9848 0)
       (effects (font (size 1.27 1.27)) hide)
     )
@@
       (effects (font (size 1.27 1.27)) hide)
     )
-    (property "Distributor Part #" "" (at 163.83 106.68 0)
-      (effects (font (size 1.27 1.27)) hide)
-    )
-    (property "Part #" "" (at 163.83 106.68 0)
-      (effects (font (size 1.27 1.27)) hide)
-    )
-    (property "Unit Price" "" (at 163.83 106.68 0)
+    (property "Distributor Part #" "HS351-ND" (at 163.83 106.68 0)
+      (effects (font (size 1.27 1.27)) hide)
+    )
+    (property "Part #" "531002B02500G" (at 163.83 106.68 0)
+      (effects (font (size 1.27 1.27)) hide)
+    )
+    (property "Unit Price" "1.55" (at 163.83 106.68 0)
       (effects (font (size 1.27 1.27)) hide)
     )
@@
   (symbol (lib_id "Connector:TestPoint") (at 100.33 74.93 0) (unit 1)
     (in_bom yes) (on_board yes) (dnp no) (fields_autoplaced)
-    (property "Reference" "TP6" (at 102.87 70.993 0)
-      (effects (font (size 1.27 1.27)) (justify left))
-    )
-    (property "Value" "TestPoint" (at 102.87 73.533 0)
+    (property "Reference" "TP6" (at 102.87 70.358 0)
+      (effects (font (size 1.27 1.27)) (justify left))
+    )
+    (property "Value" "4952" (at 102.87 72.898 0)
       (effects (font (size 1.27 1.27)) (justify left))
     )
@@
       (effects (font (size 1.27 1.27)) hide)
     )
-    (property "Distributor Part #" "" (at 100.33 74.93 0)
-      (effects (font (size 1.27 1.27)) hide)
-    )
-    (property "Part #" "" (at 100.33 74.93 0)
-      (effects (font (size 1.27 1.27)) hide)
-    )
-    (property "Unit Price" "" (at 100.33 74.93 0)
+    (property "Distributor Part #" "36-4952-ND" (at 100.33 74.93 0)
+      (effects (font (size 1.27 1.27)) hide)
+    )
+    (property "Part #" "4952" (at 100.33 74.93 0)
+      (effects (font (size 1.27 1.27)) hide)
+    )
+    (property "Unit Price" "0.26" (at 100.33 74.93 0)
       (effects (font (size 1.27 1.27)) hide)
     )
@@
       (effects (font (size 1.27 1.27)) hide)
     )
-    (property "Distributor Part #" "" (at 110.49 86.36 0)
-      (effects (font (size 1.27 1.27)) hide)
-    )
-    (property "Part #" "" (at 110.49 86.36 0)
-      (effects (font (size 1.27 1.27)) hide)
-    )
-    (property "Unit Price" "" (at 110.49 86.36 0)
-      (effects (font (size 1.27 1.27)) hide)
-    )
+    (property "Distributor Part #" "LMC6484IN/NOPB-ND" (at 110.49 86.36 0)
+      (effects (font (size 1.27 1.27)) hide)
+    )
+    (property "Part #" "LMC6484IN/NOPB" (at 110.49 86.36 0)
+      (effects (font (size 1.27 1.27)) hide)
+    )
+    (property "Unit Price" "2.83" (at 110.49 86.36 0)
+      (effects (font (size 1.27 1.27)) hide)
+    )

Commit message: changed crossover resistor to 330
Parts:
- R9: value 1k -> 330
Changed lines of the file:
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@@
       (effects (font (size 1.27 1.27)))
     )
-    (property "Value" "1k" (at 147.32 87.63 90)
+    (property "Value" "330" (at 148.59 87.63 90)
       (effects (font (size 1.27 1.27)))
     )

Commit message: debug and misc
Parts:
- R6: value 10k -> 100k
- R7: value 10k -> 47k
Changed lines of the file:
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@@
   )
   (symbol (lib_id "Device:R_US") (at 144.78 132.08 90) (unit 1)
-    (in_bom yes) (on_board yes) (dnp no) (fields_autoplaced)
+    (in_bom yes) (on_board yes) (dnp no)
     (property "Reference" "R6" (at 144.78 127 90)
       (effects (font (size 1.27 1.27)))
     )
-    (property "Value" "10k" (at 144.78 129.54 90)
+    (property "Value" "100k" (at 144.78 129.54 90)
       (effects (font (size 1.27 1.27)))
     )
@@
   )
   (symbol (lib_id "Device:R_US") (at 101.6 137.16 0) (unit 1)
-    (in_bom yes) (on_board yes) (dnp no) (fields_autoplaced)
-    (property "Reference" "R7" (at 104.14 136.525 0)
+    (in_bom yes) (on_board yes) (dnp no)
+    (property "Reference" "R7" (at 102.87 135.89 0)
       (effects (font (size 1.27 1.27)) (justify left))
     )
-    (property "Value" "10k" (at 104.14 139.065 0)
+    (property "Value" "47k" (at 102.87 138.43 0)
       (effects (font (size 1.27 1.27)) (justify left))
     )
